Commit message: fix(nav2_bringup): urdf check ok

File: nav2_bringup/bringup/urdf/beetle/accessories/intel_realsense.urdf.xacro (robot description, xacro)
@@ -24,5 +24,5 @@
       <gazebo reference="${frame}">
         <turnGravityOff>true</turnGravityOff>
-        <sensor type="depth" name="${prefix}_realsense_depth">
+        <sensor type="depth" name="realsense_depth">
           <update_rate>${update_rate}</update_rate>
           <camera>
@@ -68,5 +68,5 @@
       </gazebo>
     </xacro:macro>
-    <link name="${prefix}_realsense_lens">
+    <link name="realsense_lens">
       <visual>
         <!--
@@ -82,15 +82,15 @@
       </visual>
     </link>
-    <joint type="fixed" name="${prefix}_realsense_lens_joint">
+    <joint type="fixed" name="realsense_lens_joint">
       <origin xyz="0 0 0" rpy="0 0 0" />
       <parent link="${parent_link}" />
-      <child link="${prefix}_realsense_lens" />
+      <child link="realsense_lens" />
     </joint>
-    <joint type="fixed" name="${prefix}_realsense_joint">
+    <joint type="fixed" name="realsense_joint">
       <origin xyz="0.025 0 0" rpy="0 0 0" />
-      <parent link="${prefix}_realsense_lens" />
-      <child link="${prefix}_realsense" />
+      <parent link="realsense_lens" />
+      <child link="realsense" />
     </joint>
-    <xacro:intel_realsense frame="${prefix}_realsense" topic="${topic}"/>
+    <xacro:intel_realsense frame="realsense" topic="${topic}"/>
   </xacro:macro>
 </robot>

File: nav2_bringup/bringup/urdf/beetle/accessories/sensor_arch.urdf.xacro (robot description, xacro)
@@ -3,5 +3,5 @@
     <xacro:macro name="sensor_arch" params="prefix parent size:=510 *origin">
         <!-- Spawn the sensor arch link -->
-        <link name="${prefix}sensor_arch_mount_link">
+        <link name="sensor_arch_mount_link">
              <origin xyz="0 0 0" rpy="0 0 0"/>
              <visual>
@@ -18,8 +18,8 @@
         </link>
         <!-- Attach the sensor arch to the top plate -->
-        <joint name="${prefix}sensor_arch_mount" type="fixed">
+        <joint name="sensor_arch_mount" type="fixed">
              <xacro:insert_block name="origin"/>
              <parent link="${parent}"/>
-             <child link="${prefix}sensor_arch_mount_link"/>
+             <child link="sensor_arch_mount_link"/>
         </joint>
     </xacro:macro>

File: nav2_bringup/bringup/urdf/beetle/accessories/sick_lms1xx_mount.urdf.xacro (robot description, xacro)
@@ -28,5 +28,5 @@
   <xacro:include filename="$(find lms1xx)/urdf/sick_lms1xx.urdf.xacro" />
   <xacro:macro name="sick_lms1xx_mount" params="prefix">
-    <link name="${prefix}_laser_mount">
+    <link name="laser_mount">
       <visual>
         <origin xyz="0 0 0" rpy="0 0 ${-M_PI/2}" />
@@ -43,9 +43,9 @@
       </collision>
     </link>
-    <joint name="${prefix}_laser_joint" type="fixed">
+    <joint name="laser_joint" type="fixed">
       <!-- This offset is from the base of the bracket to the LIDAR's focal point. -->
       <origin xyz="0.0352 0 0.0566" rpy="${M_PI} 0 0" />
-      <parent link="${prefix}_laser_mount" />
-      <child link="${prefix}_laser" />
+      <parent link="laser_mount" />
+      <child link="laser" />
     </joint>
   </xacro:macro>

File: nav2_bringup/bringup/urdf/beetle/base.xacro (robot description, xacro)
@@ -1,7 +1,8 @@
 <?xml version="1.0"?>
-<robot xmlns:xacro="http://ros.org/wiki/xacro">
+<robot xmlns:xacro="http://ros.org/wiki/xacro" name="base">
   <xacro:arg name="laser_enabled" default="1" />
   <xacro:arg name="laser_xyz" default="0.2206 0.0 0.00635" />
   <xacro:arg name="laser_rpy" default="0.0 0.0 0.0" />
+  <xacro:property name="laser_z_offset" value="0.1" />
   <xacro:arg name="realsense_enabled" default="0" />
   <xacro:arg name="realsense_xyz" default="0 0 0" />
@@ -33,5 +34,5 @@
     <xacro:property name="wheel_radius" value="0.1651" />
     <!-- Base link is the center of the robot's bottom plate -->
-    <link name="${prefix}base_link">
+    <link name="base_link">
       <visual>
         <origin xyz="0 0 0" rpy="0 0 0" />
@@ -54,12 +55,12 @@
     </link>
     <!-- Base footprint is on the ground under the robot -->
-    <link name="${prefix}base_footprint"/>
-    <joint name="${prefix}base_footprint_joint" type="fixed">
+    <link name="base_footprint"/>
+    <joint name="base_footprint_joint" type="fixed">
       <origin xyz="0 0 ${wheel_vertical_offset - wheel_radius}" rpy="0 0 0" />
-      <parent link="${prefix}base_link" />
-      <child link="${prefix}base_footprint" />
+      <parent link="base_link" />
+      <child link="base_footprint" />
     </joint>
     <!-- Inertial link stores the robot's inertial information -->
-    <link name="${prefix}inertial_link">
+    <link name="inertial_link">
       <inertial>
         <mass value="46.034" />
@@ -68,77 +69,62 @@
       </inertial>
     </link>
-    <joint name="${prefix}inertial_joint" type="fixed">
+    <joint name="inertial_joint" type="fixed">
       <origin xyz="0 0 0" rpy="0 0 0" />
-      <parent link="${prefix}base_link" />
-      <child link="${prefix}inertial_link" />
+      <parent link="base_link" />
+      <child link="inertial_link" />
     </joint>
     <!-- IMU Link-->
     <!-- Can be modified with environment variables in /etc/ros/setup.bash -->
-    <link name="${prefix}imu_link"/>
-    <joint name="${prefix}imu_joint" type="fixed">
+    <link name="imu_link"/>
+    <joint name="imu_joint" type="fixed">
       <origin xyz="0 0 0" rpy="0 0 0" />
-      <parent link="${prefix}base_link" />
-      <child link="${prefix}imu_link" />
+      <parent link="base_link" />
+      <child link="imu_link" />
     </joint>
     <!-- GPS Link-->
     <!-- Can be modified with environment variables in /etc/ros/setup.bash -->
-    <link name="${prefix}gps_link"/>
-    <joint name="${prefix}gps_joint" type="fixed">
+    <link name="gps_link"/>
+    <joint name="gps_joint" type="fixed">
       <origin xyz="0 0 0" rpy="0 0 0" />
-      <parent link="${prefix}base_link" />
-      <child link="${prefix}gps_link" />
+      <parent link="base_link" />
+      <child link="gps_link" />
     </joint>
     <!-- LASER Link-->
-    <link name="${prefix}base_scan">
+    <link name="base_scan">
       <inertial>
         <origin xyz="-0.052 0 0.111" rpy="0 0 0" />
-        <inertia>
-          <ixx>0.001</ixx>
-          <ixy>0.000</ixy>
-          <ixz>0.000</ixz>
-          <iyy>0.001</iyy>
-          <iyz>0.000</iyz>
-          <izz>0.001</izz>
-        </inertia>
-        <mass>0.125</mass>
+        <inertia ixx="0.001" ixy="0.000" ixz="0.000" iyy="0.001" iyz="0.000" izz="0.001" />
+        <mass value="0.125"/>
       </inertial>
       <collision name="lidar_sensor_collision">
         <origin xyz="-0.052 0 0.111" rpy="0 0 0" />
         <geometry>
-          <cylinder>
-            <radius>0.0508</radius>
-            <length>0.055</length>
-          </cylinder>
+          <cylinder radius="0.0508" length="0.055" />
         </geometry>
       </collision>
-      <visual name="lidar_sensor_visual">
-        <origin xyz="-0.064 0 ${base_z_size}+0.1" rpy="0 0 0" />
+      <visual>
+        <origin xyz="-0.064 0 0.35" rpy="0 0 0" />
         <geometry>
-          <mesh>
-            <uri>model://turtlebot3_waffle/meshes/lds.dae</uri>
-            <scale>0.001 0.001 0.001</scale>
-          </mesh>
+          <mesh filename="package://nav2_bringup/meshes/accessories/lms1xx_mount.dae" />
         </geometry>
       </visual>
     </link>
     <joint name="lidar_joint" type="fixed">
-      <parent>base_link</parent>
-      <child>base_scan</child>
-      <pose>-0.064 0 0.121 0 0 0</pose>
-      <axis>
-        <xyz>0 0 1</xyz>
-      </axis>
+      <origin xyz="-0.064 0 0.121" rpy="0 0 0" />
+      <parent link="base_link" />
+      <child link="base_scan" />
+      <axis xyz="0 0 1" />
     </joint>
     <!-- beetle wheel macros -->
-    <xacro:wheel wheel_prefix="${prefix}front_left">
+    <xacro:wheel wheel_prefix="front_left">
       <origin xyz="${wheelbase/2} ${track/2} ${wheel_vertical_offset}" rpy="0 0 0" />
     </xacro:wheel>
-    <xacro:wheel wheel_prefix="${prefix}front_right">
+    <xacro:wheel wheel_prefix="front_right">
       <origin xyz="${wheelbase/2} ${-track/2} ${wheel_vertical_offset}" rpy="0 0 0" />
     </xacro:wheel>
-    <xacro:wheel wheel_prefix="${prefix}rear_left">
+    <xacro:wheel wheel_prefix="rear_left">
       <origin xyz="${-wheelbase/2} ${track/2} ${wheel_vertical_offset}" rpy="0 0 0" />
     </xacro:wheel>
-    <xacro:wheel wheel_prefix="${prefix}rear_right">
+    <xacro:wheel wheel_prefix="rear_right">
       <origin xyz="${-wheelbase/2} ${-track/2} ${wheel_vertical_offset}" rpy="0 0 0" />
     </xacro:wheel>

File: nav2_bringup/bringup/urdf/beetle/beetle.urdf (robot description, URDF)
Before this commit: robot beetle_sensor, 10 links, 9 joints
Links:
- link base_scan: mass None -> 0.125; geometry collision cylinder length=0.055 radius=0.0508; visual mesh filename=package://nav2_bringup/meshes/accessories/lms1xx_mount.dae
Joints:
- joint lidar_joint: axis  -> 0 0 1; child  -> base_scan; origin (none) -> xyz=-0.064 0 0.121 rpy=0 0 0; parent  -> base_link

File: nav2_bringup/bringup/urdf/beetle/beetle.xacro (robot description, xacro)
@@ -1,4 +1,4 @@
 <?xml version="1.0"?>
-<robot xmlns:xacro="http://ros.org/wiki/xacro" name="beetle_sensor">
+<robot xmlns:xacro="http://ros.org/wiki/xacro" name="beetle">
   <!-- robot name parameter -->
   <!-- <xacro:arg name="name" default="" /> -->
@@ -22,10 +22,10 @@
       <broadcastTF>false</broadcastTF>
       <!-- output -->
-      <publish_odom>true</publish_odom>
+      <!-- <publish_odom>true</publish_odom>
       <publish_odom_tf>true</publish_odom_tf>
       <publish_wheel_tf>false</publish_wheel_tf>
       <odometry_topic>odom</odometry_topic>
       <odometry_frame>odom</odometry_frame>
-      <robot_base_frame>base_footprint</robot_base_frame>
+      <robot_base_frame>base_footprint</robot_base_frame> -->
     </plugin>
   </gazebo>

File: nav2_bringup/bringup/urdf/beetle/wheel.xacro (robot description, xacro)
@@ -1,4 +1,4 @@
 <?xml version="1.0"?>
-<robot xmlns:xacro="http://ros.org/wiki/xacro" name="beetle_wheel">
+<robot xmlns:xacro="http://ros.org/wiki/xacro" name="wheel">
   <xacro:macro name="wheel" params="wheel_prefix *joint_pose">
     <link name="${wheel_prefix}_wheel">
