Commit message: fix(ackermann sdf): ok

File: nav2_bringup/bringup/urdf/racecar/racecar.urdf (robot description, URDF)
Before this commit: robot racecar, 22 links, 21 joints
Joints:
- removed joint left_front_shock
- removed joint left_rear_shock
- removed joint right_front_shock
- removed joint right_rear_shock
- added joint left_front_w_joint: type fixed, parent chassis, child left_steering_link, origin xyz=0.1675                    0.1525                    -0.0235 rpy=0 0 0
- added joint left_rear_w_joint: type fixed, parent chassis, child left_rear_axle_carrier, origin xyz=-0.1675                    0.1525                    -0.0235 rpy=0 0 0
- added joint right_front_w_joint: type fixed, parent chassis, child right_steering_link, origin xyz=0.1675                    -0.1525                    -0.0235 rpy=0 0 0
- added joint right_rear_w_joint: type fixed, parent chassis, child right_rear_axle_carrier, origin xyz=-0.1675                    -0.1525                    -0.0235 rpy=0 0 0

File: nav2_bringup/bringup/urdf/racecar/racecar.xacro (robot description, xacro)
@@ -195,30 +195,4 @@
     </gazebo>
   </xacro:macro>
-  <!-- Shock absorber -->
-  <xacro:macro name="shock"
-               params="lr_prefix fr_prefix lr_reflect fr_reflect child">
-    <joint name="${lr_prefix}_${fr_prefix}_shock" type="prismatic">
-      <parent link="chassis"/>
-      <child link="${child}"/>
-      <origin xyz="${fr_reflect * wheelbase / 2}
-                   ${lr_reflect * ((hex_hub_dist / 2) - axle_length)}
-                   ${(wheel_travel / 2) - shock_z_offset}"/>
-      <axis xyz="0 0 -1"/>
-      <limit lower="${-wheel_travel / 2}" upper="${wheel_travel / 2}"
-             effort="${shock_eff_limit}" velocity="${shock_vel_limit}"/>
-    </joint>
-    <transmission name="${lr_prefix}_${fr_prefix}_shock_trans">
-      <type>transmission_interface/SimpleTransmission</type>
-      <joint name="${lr_prefix}_${fr_prefix}_shock">
-        <hardwareInterface>hardware_interface/EffortJointInterface</hardwareInterface>
-      </joint>
-      <actuator name="${lr_prefix}_${fr_prefix}_shock_act">
-        <!-- This hardwareInterface element exists for compatibility
-             with ROS Hydro. -->
-        <hardwareInterface>hardware_interface/EffortJointInterface</hardwareInterface>
-        <mechanicalReduction>1</mechanicalReduction>
-      </actuator>
-    </transmission>
-  </xacro:macro>
   <!-- The "wheel" macro defines an axle carrier, axle, and wheel. -->
   <xacro:macro name="wheel" params="lr_prefix fr_prefix lr_reflect">
@@ -266,10 +240,15 @@
   <xacro:macro name="front_wheel"
                params="lr_prefix fr_prefix lr_reflect fr_reflect">
-    <xacro:shock lr_prefix="${lr_prefix}" fr_prefix="${fr_prefix}"
-                 lr_reflect="${lr_reflect}" fr_reflect="${fr_reflect}"
-                 child="${lr_prefix}_steering_link"/>
     <link name="${lr_prefix}_steering_link">
       <xacro:null_inertial/>
     </link>
+    <joint name="${lr_prefix}_${fr_prefix}_w_joint" type="fixed">
+      <parent link="chassis"/>
+      <child link="${lr_prefix}_steering_link"/>
+      <origin xyz="${fr_reflect * wheelbase / 2}
+                   ${lr_reflect * ((hex_hub_dist / 2) - axle_length)}
+                   ${(wheel_travel / 2) - shock_z_offset}"
+              rpy="0 0 0"/>
+    </joint>
     <joint name="${lr_prefix}_steering_joint" type="revolute">
       <parent link="${lr_prefix}_steering_link"/>
@@ -285,9 +264,14 @@
   <xacro:macro name="rear_wheel"
                params="lr_prefix fr_prefix lr_reflect fr_reflect">
-    <xacro:shock lr_prefix="${lr_prefix}" fr_prefix="${fr_prefix}"
-                 lr_reflect="${lr_reflect}" fr_reflect="${fr_reflect}"
-                 child="${lr_prefix}_${fr_prefix}_axle_carrier"/>
     <xacro:wheel lr_prefix="${lr_prefix}" fr_prefix="${fr_prefix}"
                  lr_reflect="${lr_reflect}"/>
+    <joint name="${lr_prefix}_${fr_prefix}_w_joint" type="fixed">
+      <parent link="chassis"/>
+      <child link="${lr_prefix}_${fr_prefix}_axle_carrier"/>
+      <origin xyz="${fr_reflect * wheelbase / 2}
+                   ${lr_reflect * ((hex_hub_dist / 2) - axle_length)}
+                   ${(wheel_travel / 2) - shock_z_offset}"
+              rpy="0 0 0"/>
+    </joint>
   </xacro:macro>
   <!-- chassis for sensors -->
@@ -445,2 +429,37 @@
   <camera prefix="camera"/>
 </robot>
+      <plugin name="racecar_ackermann_drive" filename="libgazebo_ros_ackermann_drive.so">
+        <ros>
+          <!-- <namespace>/tb3</namespace> -->
+        </ros>
+        <update_rate>30</update_rate>
+        <!-- wheels -->
+        <front_left_joint>left_front_wheel_joint</front_left_joint>
+        <front_right_joint>right_front_wheel_joint</front_right_joint>
+        <rear_left_joint>left_rear_wheel_joint</rear_left_joint>
+        <rear_right_joint>right_rear_wheel_joint</rear_right_joint>
+        <left_steering_joint>left_steering_joint</left_steering_joint>
+        <right_steering_joint>right_steering_joint</right_steering_joint>
+        <!-- <steering_wheel_joint>steering_joint</steering_wheel_joint> -->
+        <!-- Max absolute steer angle for tyre in radians-->
+        <!-- Any cmd_vel angular z greater than this would be capped -->
+        <max_steer>0.6458</max_steer>
+        <!-- Max absolute steering angle of steering wheel -->
+        <max_steering_angle>7.85</max_steering_angle>
+        <!-- Max absolute linear speed in m/s -->
+        <max_speed>1.2</max_speed>
+        <!-- PID tuning -->
+        <left_steering_pid_gain>1500 0 1</left_steering_pid_gain>
+        <left_steering_i_range>0 0</left_steering_i_range>
+        <right_steering_pid_gain>1500 0 1</right_steering_pid_gain>
+        <right_steering_i_range>0 0</right_steering_i_range>
+        <linear_velocity_pid_gain>1000 0 1</linear_velocity_pid_gain>
+        <linear_velocity_i_range>0 0</linear_velocity_i_range>
+        <!-- output -->
+        <publish_odom>true</publish_odom>
+        <publish_odom_tf>true</publish_odom_tf>
+        <publish_wheel_tf>true</publish_wheel_tf>
+        <publish_distance>true</publish_distance>
+        <odometry_frame>odom</odometry_frame>
+        <robot_base_frame>base_footprint</robot_base_frame>
+      </plugin>

Commit message: fix(racecar ackermann ok): racecar ackermann ok

File: nav2_bringup/bringup/urdf/racecar/racecar.urdf (robot description, URDF)
Before this commit: robot racecar, 22 links, 21 joints
Links:
- removed link camera_link
- removed link chassis
- removed link laser_link
- removed link left_battery
- removed link left_battery_offset
- removed link left_front_axle_carrier
- removed link left_rear_axle_carrier
- removed link left_steering_link
- removed link lidar_platform_link
- removed link platform_link
- removed link right_battery
- removed link right_battery_offset
- removed link right_front_axle_carrier
- removed link right_rear_axle_carrier
- removed link right_steering_link
- added link base_scan, mass 0.125
- added link left_front_axle, mass 0.1
- added link left_steering, mass 0.1
- added link right_front_axle, mass 0.1
- added link right_steering, mass 0.1
- link base_link: mass None -> 100; geometry collision box size=0.1 0.1 0.02; visual box size=0.1 0.1 0.02
- link imu_link: mass 0.001 -> None; geometry 
- link left_front_wheel: mass 0.29 -> 1.0; geometry 
- link left_rear_wheel: mass 0.29 -> 1.0; geometry 
- link right_front_wheel: mass 0.29 -> 1.0; geometry 
- link right_rear_wheel: mass 0.29 -> 1.0; geometry 
Joints:
- removed joint base_footprint_to_base_link
- removed joint base_link_to_chassis
- removed joint camera_joint
- removed joint chassis_to_left_battery
- removed joint chassis_to_right_battery
- removed joint left_front_axle
- removed joint left_front_w_joint
- removed joint left_rear_axle
- removed joint left_rear_w_joint
- removed joint lidar_joint
- removed joint lidar_platform_joint
- removed joint offset_to_left_battery
- removed joint offset_to_right_battery
- removed joint platform_joint
- removed joint right_front_axle
- removed joint right_front_w_joint
- removed joint right_rear_axle
- removed joint right_rear_w_joint
- added joint base_joint: type fixed, parent base_footprint, child base_link, origin xyz=0 0 0.04 rpy=0 0 0
- added joint left_front_wheel_joint: type continuous, parent left_front_axle, child left_front_wheel, origin xyz=0.13 0.08 0.04 rpy=0 0 0, axis 0 1 0
- added joint left_joint: type fixed, parent base_link, child left_steering, origin xyz=0.13 0.08 0.05 rpy=0 0 0
- added joint left_rear_wheel_joint: type continuous, parent base_link, child left_rear_wheel, origin xyz=-0.13 0.08 0.04 rpy=0 0 0, axis 0 1 0
- added joint right_front_wheel_joint: type continuous, parent right_front_axle, child right_front_wheel, origin xyz=0.13 -0.08 0.04 rpy=0 0 0, axis 0 1 0
- added joint right_joint: type fixed, parent base_link, child right_steering, origin xyz=0.13 -0.08 0.05 rpy=0 0 0
- added joint right_rear_wheel_joint: type continuous, parent base_link, child right_rear_wheel, origin xyz=-0.13 -0.08 0.04 rpy=0 0 0, axis 0 1 0
- added joint scan_joint: type fixed, parent base_link, child base_scan, origin xyz=0 0 0.1 rpy=0 0 0
- joint imu_joint: origin xyz=0.16 0 0.015 rpy=0 0 0 -> xyz=0.0 0 0.04 rpy=0 0 0; parent platform_link -> base_link
- joint left_steering_joint: child left_front_axle_carrier -> left_front_axle; limit lower=-0.785398163 upper=0.785398163 effort=0.5649 velocity=4.553 -> (none); origin (none) -> xyz=0.13 0.08 0.05 rpy=0 0 0; parent left_steering_link -> left_steering; type revolute -> continuous
- joint right_steering_joint: child right_front_axle_carrier -> right_front_axle; limit lower=-0.785398163 upper=0.785398163 effort=0.5649 velocity=4.553 -> (none); origin (none) -> xyz=0.13 -0.08 0.05 rpy=0 0 0; parent right_steering_link -> right_steering; type revolute -> continuous

Commit message: fix(gazebo test): test steering

File: nav2_bringup/bringup/urdf/racecar/racecar.urdf (robot description, URDF)
Before this commit: robot racecar, 12 links, 11 joints
Links:
- added link left_brush, mass 1.0
- added link right_brush, mass 1.0
Joints:
- added joint left_brush_joint: type fixed, parent base_link, child left_brush, origin xyz=0.16 0.1 0.01 rpy=0 0 0
- added joint right_brush_joint: type fixed, parent base_link, child right_brush, origin xyz=0.16 -0.1 0.01 rpy=0 0 0

Commit message: fix(gazebo test): test

File: nav2_bringup/bringup/urdf/racecar/racecar.urdf (robot description, URDF)
Before this commit: robot racecar, 14 links, 13 joints
Links:
- removed link left_front_axle
- removed link left_front_wheel
- removed link left_steering
- removed link right_front_axle
- removed link right_front_wheel
- removed link right_steering
Joints:
- removed joint left_front_wheel_joint
- removed joint left_joint
- removed joint left_steering_joint
- removed joint right_front_wheel_joint
- removed joint right_joint
- removed joint right_steering_joint

Commit message: fix(gazebo model): ei

File: nav2_bringup/bringup/urdf/racecar/racecar.urdf (robot description, URDF)
Before this commit: robot racecar, 8 links, 7 joints
Links:
- added link left_front_axle, mass 0.1
- added link left_front_wheel, mass 1.0
- added link left_steering, mass 0.1
- added link right_front_axle, mass 0.1
- added link right_front_wheel, mass 1.0
- added link right_steering, mass 0.1
Joints:
- added joint left_front_wheel_joint: type continuous, parent left_front_axle, child left_front_wheel, origin xyz=0.13 0.08 0.04 rpy=0 0 0, axis 0 1 0
- added joint left_joint: type fixed, parent base_link, child left_steering, origin xyz=0.13 0.08 0.05 rpy=0 0 0
- added joint left_steering_joint: type continuous, parent left_steering, child left_front_axle, origin xyz=0.13 0.08 0.05 rpy=0 0 0, axis 0 0 1
- added joint right_front_wheel_joint: type continuous, parent right_front_axle, child right_front_wheel, origin xyz=0.13 -0.08 0.04 rpy=0 0 0, axis 0 1 0
- added joint right_joint: type fixed, parent base_link, child right_steering, origin xyz=0.13 -0.08 0.05 rpy=0 0 0
- added joint right_steering_joint: type continuous, parent right_steering, child right_front_axle, origin xyz=0.13 -0.08 0.05 rpy=0 0 0, axis 0 0 1
